File: minima.sch (KiCad schematic (older format))
At the start: 9 parts, among them J1 output, J2 input, J3 powersupply

Commit message: Switching to single sch sheet 1
Parts:
- added C1, C10: 15p, Capacitor_THT:C_Disc_D3.4mm_W2.1mm_P2.50mm, symbol Device:C
- added C11, C12: 2m2, Capacitor_THT:CP_Radial_D16.0mm_P7.50mm, symbol Device:CP1
- added C13: 220p, Capacitor_THT:C_Disc_D4.3mm_W1.9mm_P5.00mm, symbol Device:C
- added C14: 2n2, Capacitor_THT:C_Disc_D4.3mm_W1.9mm_P5.00mm, symbol Device:C
- added C2: 220n, Capacitor_THT:C_Rect_L7.0mm_W3.5mm_P5.00mm, symbol Device:C
- added C3: 100n, Capacitor_THT:C_Disc_D5.1mm_W3.2mm_P5.00mm, symbol Device:C
- added C4, C7: 470u, Capacitor_THT:CP_Radial_D8.0mm_P3.50mm, symbol Device:CP1
- added C5, C8: 100n, Capacitor_THT:C_Rect_L7.0mm_W3.5mm_P5.00mm, symbol Device:C
- added C6, C9: 100u, Capacitor_THT:CP_Radial_D8.0mm_P3.50mm, symbol Device:CP1
- added D1, D2: 1N5404, Diode_THT:D_DO-201AD_P12.70mm_Horizontal, symbol Diode:1N5404
- added L1: 2u, Inductor_THT:L_Axial_L12.0mm_D5.0mm_P15.24mm_Horizontal_Fastron_MISC, symbol Device:L
- added R1, R9: 1k6, Resistor_THT:R_Axial_DIN0207_L6.3mm_D2.5mm_P7.62mm_Horizontal, symbol Device:R
- added R10, R11: 100, Resistor_THT:R_Axial_DIN0207_L6.3mm_D2.5mm_P7.62mm_Horizontal, symbol Device:R
- added R12: 100k, Resistor_THT:R_Axial_DIN0207_L6.3mm_D2.5mm_P7.62mm_Horizontal, symbol Device:R
- added R13: 10, Resistor_THT:R_Axial_DIN0207_L6.3mm_D2.5mm_P10.16mm_Horizontal, symbol Device:R
- added R2, R6: 4.7, Resistor_THT:R_Axial_DIN0411_L9.9mm_D3.6mm_P15.24mm_Horizontal, symbol Device:R
- added R3: 10, Resistor_THT:R_Axial_DIN0411_L9.9mm_D3.6mm_P15.24mm_Horizontal, symbol Device:R
- added R4, R7: 499, Resistor_THT:R_Axial_DIN0207_L6.3mm_D2.5mm_P10.16mm_Horizontal, symbol Device:R
- added R5, R8: 7k5, Resistor_THT:R_Axial_DIN0207_L6.3mm_D2.5mm_P10.16mm_Horizontal, symbol Device:R
- added U1: LM1875, Package_TO_SOT_THT:TO-220-5_P3.4x3.7mm_StaggerOdd_Lead3.8mm_Vertical, symbol Amplifier_Audio:LM1875
Connections:
- net labels added: VCC, VEE, inp, sgnd, spkhot
- wire segments 16 -> 105
Other:
- note added: "Fz=1.6e6\nFp=6.6e6"
- note added: "Put R10 and C13 right next to\ninput connector. The return\nground should be at the connector\nside."
- note added: "Put R3 and C3 right next to output \nconnector. Also, the return ground \nshould be at the connector side."
- moved on the sheet: J1, J3

Commit message: Removed sheets
Parts:
- R1: footprint Resistor_THT:R_Axial_DIN0207_L6.3mm_D2.5mm_P7.62mm_Horizontal -> Resistor_THT:R_Axial_DIN0207_L6.3mm_D2.5mm_P10.16mm_Horizontal
- R13: renamed from R9; footprint Resistor_THT:R_Axial_DIN0207_L6.3mm_D2.5mm_P7.62mm_Horizontal -> Resistor_THT:R_Axial_DIN0207_L6.3mm_D2.5mm_P10.16mm_Horizontal
- R4: renamed from R10; footprint Resistor_THT:R_Axial_DIN0207_L6.3mm_D2.5mm_P7.62mm_Horizontal -> Resistor_THT:R_Axial_DIN0207_L6.3mm_D2.5mm_P10.16mm_Horizontal
- R5: renamed from R11; footprint Resistor_THT:R_Axial_DIN0207_L6.3mm_D2.5mm_P7.62mm_Horizontal -> Resistor_THT:R_Axial_DIN0207_L6.3mm_D2.5mm_P10.16mm_Horizontal
- R8: renamed from R12; footprint Resistor_THT:R_Axial_DIN0207_L6.3mm_D2.5mm_P7.62mm_Horizontal -> Resistor_THT:R_Axial_DIN0207_L6.3mm_D2.5mm_P10.16mm_Horizontal
- renumbered C6 to C10, C5 to C11, C9 to C13, C8 to C14, C13 to C5, C14 to C6, C10 to C8, C11 to C9, J2 to J1, J1 to J2, R7 to R10, R8 to R11, R13 to R12, R4 to R6, R5 to R7, R6 to R9
