File: minima_amp/minima.sch (KiCad schematic (older format))
At the start: 40 parts, among them J1 input, J2 output, J3 powersupply, U1 LM1875

Commit message: WIP: Component routing & placement
Parts:
- C1, C5: Vendor Farnel:1100498 -> Farnel: 1100498
- C10, C7: Vendor Farnell:2346269 -> Farnell: 2346269
- C11, C8: Vendor Farnell:1890265 -> Farnell: 1890265
- C2: Vendor Farnell:1890146 -> Farnell: 1890146
- C3, C4: Vendor Farnell:1144610 -> Farnell: 1144610
- C6, C9: Vendor Farnell:2346272 -> Farnell: 2346272
- Clp1: Vendor Farnell:1100515 -> Farnell: 1100515
- Czi1: Vendor Farnell:1100508 -> Farnell: 1100508
- Czo1: Vendor Farnell:1100408 -> Farnell: 1100408
- D1, D2: Vendor Farnell:9556141 -> Farnell: 9556141
- J3: Vendoe Farnell: 3913089 -> (none); Vendor (none) -> Farnell: 3913089
- R1, R9: Vendor Farnell:2329892 -> Farnell: 2329892
- R2, Rd1: Vendor Farnell:2614544 -> Farnell: 2614544
- R3, R6: Vendor Farnell:2330163 -> Farnell: 2330163
- R4, R7: Vendor Farnell:2330223 -> Farnell: 2330223
- R5: Vendor Farnell:2329853 -> Farnell: 2329853
- R8: Vendor Farnell:2329993 -> Farnell: 2329993
- Rlp1, Rzi1: Vendor Farnell:2329854 -> Farnell: 2329854
- Rzo1: Vendor Farnell:2614526 -> Farnell: 2614526
- U1: Vendor Farnell:1468913 -> Farnell: 1468913

Commit message: Added comment about matching connector
Changed lines of the file:
@@
 	1    0    0    1
 $EndComp
-Text Notes 8500 2550 0    50   ~ 0
+Text Notes 8500 4600 0    50   ~ 0
 Put Rzo and Czo right next to output \nconnector. Also, the return ground \nshould be at the connector side.
 Wire Wire Line
@@
 	7750 3800 9700 3800
 Wire Notes Line
-	8450 2250 10000 2250
+	10000 4300 10000 4650
 Wire Notes Line
-	10000 2250 10000 2600
+	8450 4650 8450 4300
 Wire Notes Line
-	8450 2600 8450 2250
-Wire Notes Line
-	7400 2600 10000 2600
+	8450 4650 10000 4650
 Wire Notes Line
 	1700 5400 2950 5400
@@
 Wire Wire Line
 	7200 4500 7200 4400
+Wire Notes Line
+	7450 4300 10000 4300
 $EndSCHEMATC

Commit message: feat: simpler schematic
Signed-off-by: Nenad Radulovic <nenad.b.radulovic@gmail.com>
Parts:
- removed C1, C5: 15p, Capacitor_THT:C_Disc_D3.4mm_W2.1mm_P2.50mm, symbol Device:C
- removed C10: 100u, Capacitor_THT:CP_Radial_D8.0mm_P3.50mm, symbol Device:CP1
- removed C6, C9: 2m2, Capacitor_THT:CP_Radial_D16.0mm_P7.50mm, symbol Device:CP1
- removed Czo1: 100n, Capacitor_THT:C_Disc_D5.1mm_W3.2mm_P5.00mm, symbol Device:C
- removed R1, R9: 1k6, Resistor_THT:R_Axial_DIN0207_L6.3mm_D2.5mm_P10.16mm_Horizontal, symbol Device:R
- removed Rzo1: 10, Resistor_THT:R_Axial_DIN0411_L9.9mm_D3.6mm_P15.24mm_Horizontal, symbol Device:R
- added C4, C7, C8: 220u, Capacitor_THT:CP_Radial_D10.0mm_P5.00mm, symbol Device:CP1
- C5: renamed from C7; value 100u -> 220u; footprint Capacitor_THT:CP_Radial_D8.0mm_P3.50mm -> Capacitor_THT:CP_Radial_D10.0mm_P5.00mm
- R1: renamed from R3; value 499 -> 200
- R2: renamed from R4; value 7k5 -> 3k6
- R4: renamed from R6; value 499 -> 200
- R5: renamed from R7; value 7k5 -> 3k6
- renumbered C3 to C1, C4 to C3, C8 to C6, C11 to C9, R5 to R3, R2 to R6, R8 to R7
Connections:
- net GNDPWR: now also C4.2, C7.1, C8.1
- net VCC: now also C4.1
- net VEE: now also C7.2, C8.2
Other:
- note removed: "Put Rzo and Czo right next to output \nconnector. Also, the return ground \nshould be at the connector side."
